File: circuitry/psx-mem.kicad_pcb (KiCad board)
At the start: 2 copper layers, 36.2 x 25 mm, 30 parts, among them J2 Conn_01x06, U1 PFS154-S16, U2 ZD25WQ16C

Commit message: Schematic and layout completed.
Parts:
- removed C3: 47µF, Capacitor_SMD:C_0805_2012Metric_Pad1.18x1.45mm_HandSolder
- removed D1, D2, D3, D4: LED_Filled, LED_SMD:LED_0805_2012Metric_Pad1.15x1.40mm_HandSolder
- removed R2, R3, R4, R5: 1kΩ, Resistor_SMD:R_0805_2012Metric_Pad1.20x1.40mm_HandSolder
- added LS1: Speaker_Crystal, PSX_Memory:BUZ-SMD_4P-L7.5-W7.5-BR, F.Cu at (165.2, 103.8)
- added Q1: BC847, Package_TO_SOT_SMD:SOT-23-3, F.Cu at (159.2, 101.5)
- added Q2: BC847, Package_TO_SOT_SMD:SOT-23-3, F.Cu at (159.2, 106.0)
- added R1: 220Ω, Resistor_SMD:R_0805_2012Metric, F.Cu at (156.6, 108.9)
- added TP13: TestPoint, TestPoint:TestPoint_Pad_D1.0mm, F.Cu at (154.9, 96.8)
- C1, C2: value 100nF -> 10µF; footprint Capacitor_SMD:C_0805_2012Metric_Pad1.18x1.45mm_HandSolder -> Capacitor_SMD:C_0805_2012Metric
- J2: value Conn_01x06 -> Conn_01x03; footprint PSX_MEM:Debug_2x03_P2.54mm -> PSX_Memory:TestPoint_UPDI
- TP1, TP10, TP11, TP12, TP2, TP3, TP4, TP5, TP6, TP7, TP8, TP9: footprint PSX_MEM:TestPoint -> TestPoint:TestPoint_Pad_D1.0mm
- U1: value PFS154-S16 -> ATtiny404-SS; footprint Package_SO:SOIC-16_3.9x9.9mm_P1.27mm -> Package_SO:SOIC-14_3.9x8.7mm_P1.27mm
- moved TP8 28.5 mm to (140.0, 104.2)
- moved TP11 25.9 mm to (141.5, 105.2)
- moved TP10 24.3 mm to (141.5, 103.2)
- moved TP7 12.6 mm to (152.7, 96.8)
- moved TP3 12.6 mm to (165.2, 96.8)
- moved U2 11.2 mm to (154.8, 103.2)
- moved TP2 10.3 mm to (157.2, 96.8)
- moved C2 10.1 mm to (154.5, 108.9), turned to -90 degrees
- moved TP12 8.06 mm to (170.8, 103.2)
- moved TP4 8.00 mm to (146.9, 96.8)
- moved TP9 7.05 mm to (170.8, 105.2)
- moved J2 5.82 mm to (144.5, 108.8), turned to 0 degrees
- moved TP5 5.70 mm to (162.9, 96.8)
- moved TP6 4.60 mm to (167.6, 96.8)
- moved C1 4.15 mm to (152.4, 108.9), turned to -90 degrees
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Connections:
- J2 pad 2: /PCK -> Net-(J2-Pin_2)
- J2 pad 3: /VPP -> GND
- TP10 pad 1: /SCLK -> /MISO
- TP11 pad 1: /MISO -> /MOSI
- TP12 pad 1: /MOSI -> Net-(Q1-B)
- TP2 pad 1: /CMD -> VDD
- TP3 pad 1: +7.5V -> /CLK
- TP4 pad 1: GND -> /CMD
- TP5 pad 1: VDD -> /~{ATT}
- TP6 pad 1: /~{ATT} -> /~{ACK}
- TP7 pad 1: /CLK -> +7.5V
- TP8 pad 1: /~{ACK} -> /~{CS}
- TP9 pad 1: /~{CS} -> /SCLK
- U1 pad 1: /MISO -> VDD
- U1 pad 10: /~{ACK} -> Net-(J2-Pin_2)
- U1 pad 11: /CLK -> /MOSI
- U1 pad 12: GND -> /MISO
- U1 pad 13: /~{ATT} -> /SCLK
- U1 pad 14: /CMD -> GND
- U1 pad 2: /~{CS} -> Net-(U1-PA4)
- U1 pad 3: /SCLK -> unconnected-(U1-PA5-Pad3)
- U1 pad 4: /MOSI -> /~{ACK}
- U1 pad 5: VDD -> /~{ATT}
- U1 pad 6: unconnected-(U1-PA7/X1-Pad6) -> /CMD
- U1 pad 7: /PIO -> /DAT
- U1 pad 8: /VPP -> /CLK
- U1 pad 9: /PCK -> /~{CS}
Routing:
- net Net-(J2-Pin_4): track 31.6 -> 0.00 mm
- net /PCK: track 26.2 -> 0.00 mm, vias 1 -> 0
- net GND: track 63.2 -> 37.0 mm, vias 4 -> 5
- net Net-(U1-PA4): track 0.00 -> 23.7 mm
- net Net-(Q1-B): track 0.00 -> 19.4 mm
- net /PIO: track 16.1 -> 0.00 mm, vias 1 -> 0
- net /VPP: track 15.8 -> 0.00 mm, vias 1 -> 0
- net Net-(D1-K): track 9.96 -> 0.00 mm
- net /CLK: track 21.3 -> 30.9 mm
- net /MISO: track 27.9 -> 19.6 mm
- net Net-(D2-K): track 7.67 -> 0.00 mm
- net VDD: track 63.2 -> 55.9 mm, vias 7 -> 5
- net Net-(D4-K): track 7.03 -> 0.00 mm
- net Net-(D3-K): track 6.84 -> 0.00 mm
- net Net-(J2-Pin_2): track 0.00 -> 3.45 mm
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Other:
- board size 36.2 x 25 mm -> 36.2 x 22.5 mm
- board text added: "PSX Memory Card v1.1"
- board text removed: "A"
- board text removed: "B"
- board text removed: "C"
- board text removed: "D"
- board text removed: "E"
- board text removed: "F"
- board text removed: "G"
- board text removed: "H"
- board text removed: "I"
- board text removed: "J"
- board text removed: "K"
- board text removed: "L"
- board text removed: "M"
- board text removed: "N"
- board text removed: "O"
- board text removed: "P"
- board text removed: "PSX Memory Card v1.0"
- board text removed: "Q"
- board text removed: "R"
